File: SoftProject/SoftProject.kicad_pcb (KiCad board)
At the start: 2 copper layers, 8 parts, among them J2 Conn_01x20_Pin, J3 Conn_01x20_Pin, Q1 2N2219, Q2 2N2219, U1 ESP32-S2-WROVER, U2 AMS1117, U3 CP2102N-Axx-xQFN28

Commit message: Finished layout. Started routing.
Parts:
- removed J2: Conn_01x20_Pin, Connector_PinHeader_2.54mm:PinHeader_1x20_P2.54mm_Vertical
- added C1: 0.1uF, Capacitor_SMD:C_0402_1005Metric, F.Cu at (84.1, 59.2)
- added C10: 10uF, Capacitor_SMD:C_0805_2012Metric, F.Cu at (97.5, 104.3)
- added C11: 22pF, Capacitor_SMD:C_0402_1005Metric, F.Cu at (98.6, 87.2)
- added C12: 22pF, Capacitor_SMD:C_0402_1005Metric, F.Cu at (97.4, 87.2)
- added C13: 4.7uF, Capacitor_SMD:C_0603_1608Metric, F.Cu at (99.4, 96.4)
- added C14: 0.1uF, Capacitor_SMD:C_0402_1005Metric, F.Cu at (101.2, 96.2)
- added C15: 1uF, Capacitor_SMD:C_0402_1005Metric, F.Cu at (102.7, 103.6)
- added C2: 10uF, Capacitor_SMD:C_0805_2012Metric, F.Cu at (81.9, 59.5)
- added C3: 1uF, Capacitor_SMD:C_0402_1005Metric, F.Cu at (105.7, 58.4)
- added C4: 0.1uF, Capacitor_SMD:C_0402_1005Metric, F.Cu at (83.6, 103.8)
- added C5: 10uF, Capacitor_SMD:C_0805_2012Metric, F.Cu at (86.2, 103.8)
- added C6: 10uF, Capacitor_SMD:C_0805_2012Metric, F.Cu at (92.7, 99.8)
- added C7: 0.1uF, Capacitor_SMD:C_0402_1005Metric, F.Cu at (92.8, 96.8)
- added C8: 0.1uF, Capacitor_SMD:C_0402_1005Metric, F.Cu at (88.9, 103.8)
- added C9: 0.1uF, Capacitor_SMD:C_0402_1005Metric, F.Cu at (103.5, 105.7)
- added D1: RED, LED_SMD:LED_0603_1608Metric, F.Cu at (95.1, 95.8)
- added D3: D_Schottky, Diode_SMD:D_SOD-323, F.Cu at (94.6, 104.3)
- added G***: LOGO, LOGO, F.Cu at (105.7, 87.1)
- added H1: MountingHole, MountingHole:MountingHole_2.2mm_M2, F.Cu at (78.0, 53.3)
- added H2: MountingHole, MountingHole:MountingHole_2.2mm_M2, F.Cu at (111.0, 53.3)
- added H3: MountingHole, MountingHole:MountingHole_2.2mm_M2, F.Cu at (78.0, 115.8)
- added H4: MountingHole, MountingHole:MountingHole_2.2mm_M2, F.Cu at (111.0, 115.8)
- added J1: USB_B_Micro, Connector_USB:USB_Micro-B_Wuerth_629105150521, F.Cu at (94.6, 114.3)
- added J4: Conn_01x20_Socket, Connector_PinSocket_2.54mm:PinSocket_1x20_P2.54mm_Vertical, F.Cu at (78.0, 63.0)
- added R1: 10k, Resistor_SMD:R_0402_1005Metric, F.Cu at (105.7, 59.8)
- added R10: 47.5k, Resistor_SMD:R_0402_1005Metric, F.Cu at (104.0, 103.6)
- added R11: 10k, Resistor_SMD:R_0402_1005Metric, F.Cu at (89.3, 89.8)
- added R12: 10k, Resistor_SMD:R_0402_1005Metric, F.Cu at (90.8, 89.8)
- added R13: 10k, Resistor_SMD:R_0402_1005Metric, F.Cu at (107.8, 103.6)
- added R14: 0, Resistor_SMD:R_0402_1005Metric, F.Cu at (104.4, 93.0)
- added R15: 0, Resistor_SMD:R_0402_1005Metric, F.Cu at (105.7, 93.0)
- added R16: 0, Resistor_SMD:R_0402_1005Metric, F.Cu at (97.4, 94.9)
- added R17: 0, Resistor_SMD:R_0402_1005Metric, F.Cu at (97.4, 96.8)
- added R2: 10k, Resistor_SMD:R_0402_1005Metric, F.Cu at (93.0, 83.8)
- added R3: 5.1k, Resistor_SMD:R_0402_1005Metric, F.Cu at (92.8, 94.9)
- added R5: 0, Resistor_SMD:R_0402_1005Metric, F.Cu at (98.6, 89.4)
- added R6: 0, Resistor_SMD:R_0402_1005Metric, F.Cu at (97.4, 89.4)
- added R8: 2k, Resistor_SMD:R_0402_1005Metric, F.Cu at (106.5, 103.6)
- added R9: 22.1k, Resistor_SMD:R_0402_1005Metric, F.Cu at (105.2, 103.6)
- added SW1: SW_Push, Button_Switch_SMD:SW_SPST_B3U-1000P, F.Cu at (85.5, 112.3)
- added SW2: SW_Push, Button_Switch_SMD:SW_SPST_B3U-1000P, F.Cu at (103.6, 112.2)
- J3: value Conn_01x20_Pin -> Conn_01x20_Socket
- Q1, Q2: footprint Package_TO_SOT_THT:TO-39-3 -> Package_TO_SOT_SMD:SOT-23
- moved Q1 91.4 mm to (86.3, 89.7)
- moved Q2 84.9 mm to (93.8, 89.8), turned to 180 degrees
- moved U3 83.4 mm to (105.3, 98.0)
- moved U2 79.4 mm to (86.5, 97.9)
- moved U1 78.9 mm to (94.7, 70.1)
- moved D2 75.4 mm to (96.0, 99.8)
- moved J3 9.81 mm to (111.0, 63.0)
Connections:
- J3 pad 1: +3.3V -> GND
- J3 pad 10: /GPIO8 -> /GPIO39
- J3 pad 11: /GPIO9 -> /GPIO38
- J3 pad 12: /GPIO10 -> /GPIO37
- J3 pad 13: /GPIO11 -> /GPIO36
- J3 pad 14: /GPIO12 -> /GPIO35
- J3 pad 15: /GPIO13 -> /GPIO34
- J3 pad 16: /GPIO14 -> /GPIO33
- J3 pad 17: /GPIO15 -> /GPIO26
- J3 pad 18: /GPIO16 -> /GPIO21
- J3 pad 19: /GPIO17 -> GND
- J3 pad 2: /GPIO0 -> /CHIP_PU
- J3 pad 20: +5V -> GND
- J3 pad 3: /GPIO1 -> /GPIO46
- J3 pad 4: /GPIO2 -> /GPIO45
- J3 pad 5: /GPIO3 -> /RXD
- J3 pad 6: /GPIO4 -> /TXD
- J3 pad 7: /GPIO5 -> /GPIO42
- J3 pad 8: /GPIO6 -> /GPIO41
- J3 pad 9: /GPIO7 -> /GPIO40
- U1 pad 22: /USB_DN -> /DN
- U1 pad 23: /USB_DP -> /DP
Routing:
- net /GPIO0: track 0.00 -> 63.2 mm
- net /RXD: track 0.00 -> 46.6 mm, vias 0 -> 2
- net /TXD: track 0.00 -> 45.6 mm, vias 0 -> 2
- net /GPIO17: track 0.00 -> 37.0 mm
- net /RTS: track 0.00 -> 34.5 mm, vias 0 -> 2
- net /GPIO21: track 0.00 -> 33.4 mm, vias 0 -> 2
- net /GPIO16: track 0.00 -> 33.3 mm
- net /D-: track 0.00 -> 31.3 mm, vias 0 -> 3
- net /GPIO26: track 0.00 -> 29.7 mm, vias 0 -> 2
- net /GPIO15: track 0.00 -> 29.7 mm
- net /D+: track 0.00 -> 28.4 mm, vias 0 -> 2
- net /GPIO14: track 0.00 -> 25.8 mm
- net /GPIO33: track 0.00 -> 24.6 mm
- net /DTR: track 0.00 -> 23.3 mm, vias 0 -> 2
- net /GPIO34: track 0.00 -> 23.0 mm
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- added copper zone on In2.Cu, net +3.3V
- added copper zone on F.Cu, net GND
- added copper zone on In1.Cu, net GND
Other:
- board outline added: 38.1 x 67.6 mm
- copper layers 2 -> 4

Commit message: Finished layout and routing
Parts:
- moved C6 7.70 mm to (85.5, 102.7), turned to 180 degrees
- moved C5 6.74 mm to (91.6, 99.8), turned to 90 degrees
- moved C4 6.18 mm to (89.8, 103.8)
- moved C10 6.03 mm to (91.6, 103.4), turned to -90 degrees
- moved R9 2.62 mm to (102.6, 103.6)
- moved C15 2.59 mm to (105.3, 103.6)
- moved C14 1.02 mm to (101.2, 95.2)
- moved U2 0.79 mm to (86.5, 97.1), turned to 90 degrees
- moved C13 0.62 mm to (99.3, 95.8)
- moved C8 0.38 mm to (88.5, 103.8)
- moved G*** 0.38 mm to (105.3, 87.1)
- moved D3 0.28 mm to (94.6, 104.6)
- moved C7 0.25 mm to (92.8, 96.5)
- moved H1 0.18 mm to (78.1, 53.2)
- moved H2 0.15 mm to (110.9, 53.2)
Routing:
- net /CHIP_PU: track 15.3 -> 83.0 mm, vias 0 -> 3
- net +5V: track 0.00 -> 25.7 mm
- net GND: track 13.4 -> 36.8 mm, vias 13 -> 39
- net /GPIO0: track 63.2 -> 84.9 mm, vias 0 -> 2
- net VBUS: track 7.59 -> 26.2 mm, vias 0 -> 4
- net Net-(U3-VBUS): track 0.00 -> 6.80 mm
- net +3.3V: track 7.29 -> 13.8 mm, vias 2 -> 13
- net Net-(U3-~{SUSPEND}): track 0.00 -> 3.86 mm
- net Net-(U3-~{RST}): track 0.00 -> 3.59 mm
- net /D-: track 31.3 -> 31.9 mm
- added copper zone on F.Cu, net +3.3V
- added copper zone on F.Cu, net +5V
Other:
- board size 38.1 x 67.6 mm -> 38.1 x 67.8 mm

Commit message: Finished ESP32Board
Parts:
- SW1, SW2: footprint Button_Switch_SMD:SW_SPST_B3U-1000P -> B3U-1000P:B3U-1000P
- turned SW1 to -90 degrees
- turned SW2 to -90 degrees
Other:
- board text added: "0"
- board text added: "06/23"
- board text added: "1"
- board text added: "10"
- board text added: "11"
- board text added: "12"
- board text added: "13"
- board text added: "14"
- board text added: "15"
- board text added: "16"
- board text added: "17"
- board text added: "2"
- board text added: "21"
- board text added: "26"
- board text added: "3"
- board text added: "3.3V"
- board text added: "33"
- board text added: "34"
- board text added: "35"
- board text added: "36"
- board text added: "37"
- board text added: "38"
- board text added: "39"
- board text added: "4"
- board text added: "40"
- board text added: "41"
- board text added: "42"
- board text added: "45"
- board text added: "46"
- board text added: "5"
- board text added: "5V"
- board text added: "6"
- board text added: "7"
- board text added: "8"
- board text added: "9"
- board text added: "BOOT"
- board text added: "EN"
- board text added: "GND"
- board text added: "RXD"
- board text added: "TXD"
- board text added: "V 1.0"

Commit message: Finished and ordered PCB
Parts:
- J1: footprint Connector_USB:USB_Micro-B_Wuerth_629105150521 -> Connector_USB:USB_Micro-B_Molex-105017-0001
- moved J1 1.10 mm to (94.6, 115.4)
- moved H3 0.36 mm to (78.2, 115.6)
- moved H4 0.36 mm to (110.7, 115.6)
- moved H1 0.18 mm to (78.2, 53.3)
- moved H2 0.18 mm to (110.7, 53.3)
Connections:
- J1 pad 6: unconnected-(J1-Shield-Pad6) -> (no net)
- Q2 pad 1: /IO0_Auto -> /DTR
- Q2 pad 3: /DTR -> /IO0_Auto
Routing:
- net /DTR: track 23.5 -> 27.6 mm, vias 2 -> 0
- net /IO0_Auto: track 6.94 -> 8.67 mm
- net VBUS: track 26.2 -> 27.8 mm
- net /D-: track 31.9 -> 33.4 mm
- net /D+: track 28.7 -> 30.2 mm
- net /RTS: track 34.7 -> 35.7 mm
